File: pcb/_autosave-TP_DCI_Jordan.sch (KiCad schematic (older format))
At the start: 19 parts, among them J1 MICRO, J2 Display, SW1 SW_DIP_x03, U1 PCF8574

Commit message: revisión huella PCF8574 ok
Parts:
- U1: value PCF8574 -> PCF8574 SO16
Changed lines of the file:
@@
 P 4410 5805
 F 0 "U1" H 4105 6400 50  0000 C CNN
-F 1 "PCF8574" H 4600 6405 50  0000 C CNN
+F 1 "PCF8574 SO16" H 4760 5210 50  0000 C CNN
 F 2 "miSMD:SOIC127P1030X265-16N" H 4410 5805 50  0001 C CNN
 F 3 "http://www.nxp.com/documents/data_sheet/PCF8574_PCF8574A.pdf" H 4410 5805 50  0001 C CNN
