File: pcb/TP_DCI_Jordan.kicad_sch (KiCad schematic)
At the start: 19 parts, among them J1 MICRO, J2 LCD16x2, SW1 SW_DIP_x03, U1 PCF8574

Commit message: presentación final
Changed lines of the file:
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@@
     (stroke (width 0) (type default) (color 0 0 0 0))
   )
-  (wire (pts (xy 107.188 184.15) (xy 107.188 182.88))
+  (wire (pts (xy 107.442 181.864) (xy 107.442 180.594))
     (stroke (width 0) (type default) (color 0 0 0 0))
   )
@@
     (stroke (width 0) (type default) (color 0 0 0 0))
   )
-  (wire (pts (xy 99.06 182.88) (xy 99.06 184.15))
+  (wire (pts (xy 99.314 180.594) (xy 99.314 181.864))
     (stroke (width 0) (type default) (color 0 0 0 0))
   )
@@
     (stroke (width 0) (type default) (color 0 0 0 0))
   )
-  (wire (pts (xy 89.916 183.134) (xy 89.916 181.102))
+  (wire (pts (xy 90.17 180.848) (xy 90.17 178.816))
     (stroke (width 0) (type default) (color 0 0 0 0))
   )
@@
     (stroke (width 0) (type default) (color 0 0 0 0))
   )
-  (wire (pts (xy 99.06 184.15) (xy 107.188 184.15))
+  (wire (pts (xy 99.314 181.864) (xy 107.442 181.864))
     (stroke (width 0) (type default) (color 0 0 0 0))
   )
@@
     (pin "1")
   )
-  (symbol (lib_id "power:PWR_FLAG") (at 89.916 181.102 0) (unit 1)
-    (in_bom yes) (on_board yes)
-    (property "Reference" "#FLG0101" (id 0) (at 89.916 179.197 0)
-      (effects (font (size 1.27 1.27)) hide)
-    )
-    (property "Value" "PWR_FLAG" (id 1) (at 89.916 177.292 0))
-    (property "Footprint" "" (id 2) (at 89.916 181.102 0)
-      (effects (font (size 1.27 1.27)) hide)
-    )
-    (property "Datasheet" "~" (id 3) (at 89.916 181.102 0)
-      (effects (font (size 1.27 1.27)) hide)
-    )
-    (pin "1")
-  )
-  (symbol (lib_id "power:GND") (at 89.916 183.134 0) (unit 1)
-    (in_bom yes) (on_board yes)
-    (property "Reference" "#GND0104" (id 0) (at 89.916 189.484 0)
-      (effects (font (size 1.27 1.27)) hide)
-    )
-    (property "Value" "GND" (id 1) (at 87.884 186.944 0)
-      (effects (font (size 1.27 1.27)) (justify left))
-    )
-    (property "Footprint" "" (id 2) (at 89.916 183.134 0)
-      (effects (font (size 1.27 1.27)) hide)
-    )
-    (property "Datasheet" "" (id 3) (at 89.916 183.134 0)
-      (effects (font (size 1.27 1.27)) hide)
-    )
-    (pin "1")
-  )
-  (symbol (lib_id "power:PWR_FLAG") (at 107.188 182.88 0) (unit 1)
-    (in_bom yes) (on_board yes)
-    (property "Reference" "#FLG0102" (id 0) (at 107.188 180.975 0)
-      (effects (font (size 1.27 1.27)) hide)
-    )
-    (property "Value" "PWR_FLAG" (id 1) (at 107.188 179.07 0))
-    (property "Footprint" "" (id 2) (at 107.188 182.88 0)
-      (effects (font (size 1.27 1.27)) hide)
-    )
-    (property "Datasheet" "~" (id 3) (at 107.188 182.88 0)
-      (effects (font (size 1.27 1.27)) hide)
-    )
-    (pin "1")
-  )
-  (symbol (lib_id "power:VDD") (at 99.06 182.88 0) (unit 1)
-    (in_bom yes) (on_board yes)
-    (property "Reference" "#PWR0112" (id 0) (at 99.06 186.69 0)
-      (effects (font (size 1.27 1.27)) hide)
-    )
-    (property "Value" "VDD" (id 1) (at 99.06 179.07 0))
-    (property "Footprint" "" (id 2) (at 99.06 182.88 0)
-      (effects (font (size 1.27 1.27)) hide)
-    )
-    (property "Datasheet" "" (id 3) (at 99.06 182.88 0)
-      (effects (font (size 1.27 1.27)) hide)
-    )
+  (symbol (lib_id "power:PWR_FLAG") (at 90.17 178.816 0) (unit 1)
+    (in_bom yes) (on_board yes)
+    (property "Reference" "#FLG0101" (id 0) (at 90.17 176.911 0)
+      (effects (font (size 1.27 1.27)) hide)
+    )
+    (property "Value" "PWR_FLAG" (id 1) (at 90.17 175.006 0))
+    (property "Footprint" "" (id 2) (at 90.17 178.816 0)
+      (effects (font (size 1.27 1.27)) hide)
+    )
+    (property "Datasheet" "~" (id 3) (at 90.17 178.816 0)
+      (effects (font (size 1.27 1.27)) hide)
+    )
+    (pin "1")
+  )
+  (symbol (lib_id "power:GND") (at 90.17 180.848 0) (unit 1)
+    (in_bom yes) (on_board yes)
+    (property "Reference" "#GND0104" (id 0) (at 90.17 187.198 0)
+      (effects (font (size 1.27 1.27)) hide)
+    )
+    (property "Value" "GND" (id 1) (at 88.138 184.658 0)
+      (effects (font (size 1.27 1.27)) (justify left))
+    )
+    (property "Footprint" "" (id 2) (at 90.17 180.848 0)
+      (effects (font (size 1.27 1.27)) hide)
+    )
+    (property "Datasheet" "" (id 3) (at 90.17 180.848 0)
+      (effects (font (size 1.27 1.27)) hide)
+    )
+    (pin "1")
+  )
+  (symbol (lib_id "power:PWR_FLAG") (at 107.442 180.594 0) (unit 1)
+    (in_bom yes) (on_board yes)
+    (property "Reference" "#FLG0102" (id 0) (at 107.442 178.689 0)
+      (effects (font (size 1.27 1.27)) hide)
+    )
+    (property "Value" "PWR_FLAG" (id 1) (at 107.442 176.784 0))
+    (property "Footprint" "" (id 2) (at 107.442 180.594 0)
+      (effects (font (size 1.27 1.27)) hide)
+    )
+    (property "Datasheet" "~" (id 3) (at 107.442 180.594 0)
+      (effects (font (size 1.27 1.27)) hide)
+    )
+    (pin "1")
+  )
+  (symbol (lib_id "power:VDD") (at 99.314 180.594 0) (unit 1)
+    (in_bom yes) (on_board yes)
+    (property "Reference" "#PWR0112" (id 0) (at 99.314 184.404 0)
+      (effects (font (size 1.27 1.27)) hide)
+    )
+    (property "Value" "VDD" (id 1) (at 99.314 176.784 0))
+    (property "Footprint" "" (id 2) (at 99.314 180.594 0)
+      (effects (font (size 1.27 1.27)) hide)
+    )
+    (property "Datasheet" "" (id 3) (at 99.314 180.594 0)
+      (effects (font (size 1.27 1.27)) hide)
+    )
